File: Electronique/Audio/Audio IN_OUT/AudioToRpi.sch (KiCad schematic (older format))
At the start: 33 parts, among them J1 RJ12, J2 JACK_MONO_F, J3 JACK_MONO_F, J4 USB_OTG, K1 CONN_2, P2 CAVALIER, P3 CAVALIER, Q1 BSS123, Q2 BSS123, T1 TRANSFO2, T2 TRANSFO2, U2 FT232RL

Commit message: Audio IN_OUT MAJ
Parts:
- removed C1: CP, ~, symbol SOUND_DEB-rescue:CP
- removed C2, C3: C, ~, symbol SOUND_DEB-rescue:C
- removed C4, C5: 100n, symbol SOUND_DEB-rescue:C
- removed C6: 4,7µF, symbol SOUND_DEB-rescue:CP
- removed C7: C, symbol SOUND_DEB-rescue:C
- removed D1, D2: LED, ~, symbol SOUND_DEB-rescue:LED
- removed J1: RJ12, CEN-PCB:RJ12, symbol SOUND_DEB-rescue:RJ12
- removed J2, J3: JACK_MONO_F, ~, symbol SOUND_DEB-rescue:JACK_MONO_F
- removed J4: USB_OTG, symbol SOUND_DEB-rescue:USB_OTG
- removed K1: CONN_2, ~, symbol SOUND_DEB-rescue:CONN_2
- removed L1: BLM21A1025, symbol SOUND_DEB-rescue:INDUCTOR
- removed P2, P3: CAVALIER, ~, symbol SOUND_DEB-rescue:CAVALIER
- removed Q1, Q2: BSS123, SOT-23, symbol SOUND_DEB-rescue:BSS123
- removed R1: 220, ~, symbol SOUND_DEB-rescue:R
- removed R2: 100k, symbol SOUND_DEB-rescue:R
- removed R3: 1k, ~, symbol SOUND_DEB-rescue:R
- removed R4: 0, ~, symbol SOUND_DEB-rescue:R
- removed R5, R6: 1k, symbol SOUND_DEB-rescue:R
- removed R7: 10k, symbol SOUND_DEB-rescue:R
- removed R8: 4.7k, symbol SOUND_DEB-rescue:R
- removed RVAR1: 1k, ~, symbol SOUND_DEB-rescue:RVAR
- removed RVAR2: 1 k, ~, symbol SOUND_DEB-rescue:RVAR
- removed T1, T2: TRANSFO2, ~, symbol SOUND_DEB-rescue:TRANSFO2
- removed U2: FT232RL, SSOP-28, symbol SOUND_DEB-rescue:FT232RL
- removed U?: LTV-814, Housings_DIP:DIP-4_W7.62mm, symbol SOUND_DEB-rescue:LTV-814
Connections:
- no-connect marks 14 -> 0
Other:
- note removed: "De Sortie casque du PC\n"
- note removed: "Vers entrée ligne PC\n"
- note removed: "niveau max sans P3\nreglage par rvar2 avec P3\n"
