File: Electronique/Audio/Audio IN_OUT/Audio IN_OUT.kicad_pcb (KiCad board)
At the start: 2 copper layers, 95.2 x 95.3 mm, 47 parts, among them J1001 Conn_02x20_Odd_Even, J1002 Conn_02x20_Odd_Even, J1003 RJ12, J1004 RJ12, J1005 USB_B, J1006 USB_A, Q3001 BSS123, U3001 MC33172, U3002 MF10, U3003 TDA2003

Commit message: MAJ
Parts:
- added C3003: 10µ, Capacitor_Tantalum_SMD:CP_EIA-3216-18_Kemet-A, F.Cu at (169.2, 111.3)
- added C3010: 10µ, Capacitor_Tantalum_SMD:CP_EIA-3216-18_Kemet-A, F.Cu at (164.8, 84.8)
- added C3012: 220µ, Capacitor_SMD:CP_Elec_8x11.9, F.Cu at (150.6, 64.8)
- added C3013: 1µ, Capacitor_SMD:C_1210_3225Metric, F.Cu at (154.0, 124.5)
- added C3014: 470µ, Capacitor_SMD:CP_Elec_8x11.9, F.Cu at (150.6, 73.9)
- added C3016: 10µ, Capacitor_Tantalum_SMD:CP_EIA-3216-18_Kemet-A, F.Cu at (154.4, 112.5)
- added C3017: 1000µ, Capacitor_SMD:CP_Elec_8x11.9, F.Cu at (173.7, 60.7)
- added C3020: 10µ, Capacitor_Tantalum_SMD:CP_EIA-3216-18_Kemet-A, F.Cu at (159.7, 80.3)
- C3011: value C -> 100n
- C3015: value C -> 47n
- C3019: value C -> 0.1µ
- R3015: value R -> 100
- R3019: value R -> 47
- R3021: value R -> 220
- R3022: value R -> 2.2
- R3024: value R -> 1
- moved R3022 122.7 mm to (161.8, 75.2), turned to 90 degrees
- moved R3008 121.5 mm to (151.4, 91.9), turned to 180 degrees
- moved R3021 121.5 mm to (163.3, 75.2), turned to 270 degrees
- moved R3014 118.9 mm to (155.4, 90.4)
- moved R3015 118.7 mm to (164.0, 80.3)
- moved R3019 118.1 mm to (170.9, 68.3), turned to 180 degrees
- moved R3020 117.6 mm to (155.2, 115.1), turned to 180 degrees
- moved R3024 117.2 mm to (175.3, 67.6), turned to 90 degrees
- moved R3018 116.7 mm to (144.5, 122.4)
- moved U3001 114.5 mm to (161.3, 117.1)
- moved R3017 113.4 mm to (155.2, 116.6), turned to 180 degrees
- moved R3010 111.3 mm to (151.4, 95.0), turned to 180 degrees
- moved R3011 108.5 mm to (169.2, 91.9), turned to 180 degrees
- moved R3009 107.7 mm to (151.4, 93.5), turned to 180 degrees
- moved R3013 104.5 mm to (169.2, 95.0), turned to 180 degrees
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Connections:
- C3019 pad 1: (no net) -> /Audio-out/HP
- Q3001 pad 3: Net-(Q3001-Pad3) -> Net-(C3020-Pad2)
- R3007 pad 2: (no net) -> Net-(C3003-Pad2)
- R3015 pad 1: Net-(Q3001-Pad3) -> Net-(C3020-Pad2)
- R3015 pad 2: (no net) -> Net-(C3010-Pad1)
- R3023 pad 2: (no net) -> Net-(C3016-Pad2)
- U3003 pad 1: Net-(Q3001-Pad3) -> Net-(C3020-Pad1)
Routing:
- net Net-(C3004-Pad2): track 0.00 -> 29.2 mm
- net Net-(C3007-Pad1): track 0.00 -> 21.6 mm
- net Net-(C3015-Pad1): track 0.00 -> 20.5 mm
- net Net-(C3007-Pad2): track 0.00 -> 14.9 mm
- net Net-(C3006-Pad2): track 0.00 -> 10.3 mm
- net Net-(C3020-Pad1): track 0.00 -> 9.72 mm
- net /Audio-out/FOSC: track 0.00 -> 9.30 mm
- net +5VA: track 0.00 -> 8.02 mm
- net Net-(C3006-Pad1): track 0.00 -> 7.62 mm
- net Net-(C3020-Pad2): track 0.00 -> 6.95 mm
- net Net-(C3004-Pad1): track 0.00 -> 6.57 mm
- net /Audio-out/HP: track 0.00 -> 6.26 mm
- net Net-(C3008-Pad1): track 0.00 -> 5.24 mm
- net GND: track 0.00 -> 3.75 mm
- net Net-(R3012-Pad2): track 0.00 -> 3.57 mm
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
Commit message: CONNECTOR BOARD V2.00
Parts:
- removed J1005: USB_B, Connector_USB:USB_B_Amphenol_MUSB-D511_Vertical_Rugged
- removed J1006: USB_A, Connector_USB:USB3_A_Molex_48393-001
- added C201: 1n, Capacitor_SMD:C_0603_1608Metric, F.Cu at (164.5, 105.0)
- added C202: 100n, Capacitor_SMD:C_0603_1608Metric, F.Cu at (173.7, 108.0)
- added C203: 10µ, Capacitor_Tantalum_SMD:CP_EIA-3216-18_Kemet-A, F.Cu at (170.8, 106.4)
- added C204: 1µ, Capacitor_SMD:C_0805_2012Metric, F.Cu at (167.3, 113.6)
- added C205: C, Capacitor_SMD:C_0603_1608Metric, F.Cu at (167.9, 107.7)
- added C206: 100n, Capacitor_SMD:C_0603_1608Metric, F.Cu at (175.2, 116.5)
- added C208: 100n, Capacitor_SMD:C_0603_1608Metric, F.Cu at (184.8, 112.6)
- added C209: 100n, Capacitor_SMD:C_0603_1608Metric, F.Cu at (184.8, 115.1)
- added C210: C, Capacitor_SMD:C_0603_1608Metric, F.Cu at (180.8, 120.7)
- added D401: LED_Dual_CCA, LED_SMD:LED_LiteOn_LTST-S326, F.Cu at (214.8, 145.3)
- added L201: L, Capacitor_SMD:C_1206_3216Metric, F.Cu at (182.4, 124.3)
- added Q201: BSS123, Package_TO_SOT_SMD:SOT-23, F.Cu at (188.8, 113.7)
- added Q301: BSS123, Package_TO_SOT_SMD:SOT-23, F.Cu at (197.1, 124.2)
- added Q302: BC807W, Package_TO_SOT_SMD:SOT-23, F.Cu at (205.9, 121.2)
- added Q303: BC847, Package_TO_SOT_SMD:SOT-323_SC-70, F.Cu at (202.1, 124.1)
- added Q304: BC807W, Package_TO_SOT_SMD:SOT-23, F.Cu at (209.6, 124.7)
- added Q401: BSS123, Package_TO_SOT_SMD:SOT-23, F.Cu at (212.3, 136.5)
- added Q402: BSS123, Package_TO_SOT_SMD:SOT-23, F.Cu at (216.7, 136.5)
- added R201: 470, Resistor_SMD:R_0603_1608Metric, F.Cu at (164.4, 106.8)
- added R202: 220, Resistor_SMD:R_0603_1608Metric, F.Cu at (167.9, 105.0)
- added R203: 100k, Resistor_SMD:R_0603_1608Metric, F.Cu at (168.7, 110.0)
- added R204: 100k, Resistor_SMD:R_0603_1608Metric, F.Cu at (165.2, 110.2)
- added R205: 100k, Resistor_SMD:R_0603_1608Metric, F.Cu at (167.1, 110.0)
- added R206: 100k, Resistor_SMD:R_0603_1608Metric, F.Cu at (165.2, 113.5)
- added R207: 100k, Resistor_SMD:R_0603_1608Metric, F.Cu at (179.1, 111.8)
- added R208: 100k, Resistor_SMD:R_0603_1608Metric, F.Cu at (179.8, 115.1)
- added R209: R, Resistor_SMD:R_0603_1608Metric, F.Cu at (175.3, 118.1)
- added R210: 100k, Resistor_SMD:R_0603_1608Metric, F.Cu at (181.6, 112.6)
- added R212: 22k, Resistor_SMD:R_0603_1608Metric, F.Cu at (182.2, 118.0)
- added R213: 680, Resistor_SMD:R_0603_1608Metric, F.Cu at (184.0, 120.7)
- added R301: 100k, Resistor_SMD:R_0603_1608Metric, F.Cu at (194.1, 124.3)
- added R302: 10k, Resistor_SMD:R_0603_1608Metric, F.Cu at (194.9, 121.4)
- added R303: 1k, Resistor_SMD:R_0603_1608Metric, F.Cu at (202.1, 121.0)
- added R304: 100k, Resistor_SMD:R_0603_1608Metric, F.Cu at (216.7, 132.6)
- added R305: 1k, Resistor_SMD:R_0603_1608Metric, F.Cu at (205.8, 124.1)
- added R306: 100k, Resistor_SMD:R_0603_1608Metric, F.Cu at (212.5, 132.6)
- added R307: 47k, Resistor_SMD:R_0603_1608Metric, B.Cu at (174.4, 87.4)
- added R308: 47k, Resistor_SMD:R_0603_1608Metric, B.Cu at (179.1, 87.4)
- added R309: 47k, Resistor_SMD:R_0603_1608Metric, B.Cu at (174.4, 85.6)
- added R310: 47k, Resistor_SMD:R_0603_1608Metric, B.Cu at (179.1, 85.6)
- added R311: 47k, Resistor_SMD:R_0603_1608Metric, B.Cu at (174.4, 83.7)
- added R312: 47k, Resistor_SMD:R_0603_1608Metric, B.Cu at (179.0, 83.7)
- added R401: 1k, Resistor_SMD:R_0603_1608Metric, F.Cu at (214.8, 140.2)
- added R402: 1k, Resistor_SMD:R_0603_1608Metric, F.Cu at (216.4, 140.2)
- added U201: MC33172, Package_SO:SO-8_3.9x4.9mm_P1.27mm, F.Cu at (173.4, 112.1)
- added U301: 74LVC1G80, Package_TO_SOT_SMD:SOT-23-5, F.Cu at (170.1, 99.0)
- added U302: PCF8574, Package_SO:SOIC-16W_7.5x10.3mm_P1.27mm, F.Cu at (180.1, 85.3)
- added U303: 74HC4059, Package_SO:SOIC-24W_7.5x15.4mm_P1.27mm, F.Cu at (182.6, 98.7)
- added U304: MAX7375AXR805, Package_TO_SOT_SMD:SOT-323_SC-70, F.Cu at (179.5, 107.2)
- C3012: footprint Capacitor_SMD:CP_Elec_8x11.9 -> Capacitor_SMD:CP_Elec_6.3x5.4
- C3014: footprint Capacitor_SMD:CP_Elec_8x11.9 -> Capacitor_SMD:CP_Elec_6.3x3.9
- C3017: footprint Capacitor_SMD:CP_Elec_8x11.9 -> Capacitor_SMD:CP_Elec_6.3x4.9
- U3003: footprint CEN-PCB:TDA2003V -> Package_TO_SOT_THT:TO-220-5_P3.4x3.8mm_StaggerOdd_Lead7.13mm_TabDown
- moved J1003 31.4 mm to (188.6, 134.1)
- moved C3002 24.4 mm to (158.4, 100.6), turned to 0 degrees
- moved C3003 24.4 mm to (148.0, 99.2), turned to 90 degrees
- moved R3002 23.0 mm to (155.1, 100.6), turned to 0 degrees
- moved R3004 22.5 mm to (152.0, 100.6), turned to 180 degrees
- moved R3003 20.8 mm to (156.5, 105.0), turned to 270 degrees
- moved C3014 17.5 mm to (167.8, 70.2), turned to 180 degrees
- moved R3001 16.3 mm to (156.5, 108.6), turned to 270 degrees
- moved R3025 16.1 mm to (141.5, 115.3), turned to 0 degrees
- moved C3001 14.3 mm to (148.5, 106.9), turned to 270 degrees
- moved C3017 13.7 mm to (183.5, 70.2)
- moved U3001 13.6 mm to (152.3, 106.9), turned to 90 degrees
- moved R3018 13.1 mm to (156.5, 117.0), turned to 90 degrees
- moved C3020 12.5 mm to (152.5, 70.0), turned to 270 degrees
- moved R3016 12.3 mm to (156.5, 113.5), turned to 90 degrees
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Connections:
- net /Audio-out/FOSC renamed /Audio-out/OSC-MF10/FOSC
- C3017 pad 2: /Audio-out/HP -> /HP
- C3019 pad 1: /Audio-out/HP -> /HP
- J1001 pad 31: (no net) -> /SDA1
- J1001 pad 32: (no net) -> /SCL1
- J1003 pad 1: (no net) -> /HP
- J1003 pad 2: (no net) -> /MICRO
- J1003 pad 3: (no net) -> GND
- J1003 pad 4: (no net) -> /PTT
- J1004 pad 1: (no net) -> /BFR
- J1004 pad 2: (no net) -> /BFE
- J1004 pad 3: (no net) -> GND
- J1004 pad 4: (no net) -> /PTT
- Q3001 pad 1: (no net) -> /CMD-TX
- R3025 pad 1: (no net) -> /BFR
Routing:
- net GND: track 3.75 -> 658.2 mm, vias 0 -> 17
- net +5VA: track 8.02 -> 207.0 mm, vias 0 -> 13
- net /CMD-TX: track 0.00 -> 113.2 mm, vias 0 -> 2
- net +5VD: track 0.00 -> 108.2 mm, vias 0 -> 7
- net /PTT: track 0.00 -> 71.7 mm, vias 0 -> 3
- net /HP: track 0.00 -> 65.6 mm, vias 0 -> 1
- net /BFE: track 0.00 -> 55.3 mm, vias 0 -> 3
- net /SDA1: track 0.00 -> 47.5 mm
- net /CMD-RX: track 0.00 -> 46.3 mm, vias 0 -> 2
- net Net-(C3007-Pad2): track 14.9 -> 58.1 mm, vias 0 -> 2
- net /SCL1: track 0.00 -> 41.5 mm
- net +BATT: track 0.00 -> 26.3 mm
- net Net-(C3014-Pad1): track 0.00 -> 23.4 mm
- net /BFR: track 0.00 -> 22.9 mm, vias 0 -> 1
- net Net-(U302-Pad12): track 0.00 -> 21.9 mm, vias 0 -> 2
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