File: Electronique/Audio/Audio IN_OUT/Audio IN_OUT.sch (KiCad schematic (older format))
At the start: 6 parts, among them J1001 Conn_02x20_Odd_Even, J1002 Conn_02x20_Odd_Even

Commit message: Audio IN_OUT MAJ
Parts:
- removed J? (x2): RJ45_LED, symbol Connector:RJ45_LED
- added J1003, J1004: RJ12, Connector_RJ:RJ12_Amphenol_54601, symbol Connector:RJ12
- J1005: renamed from J?; footprint (none) -> Connector_USB:USB_B_Amphenol_MUSB-D511_Vertical_Rugged
- J1006: renamed from J?; footprint (none) -> Connector_USB:USB3_A_Molex_48393-001
Changed lines of the file:
@@
 $Descr A4 11693 8268
 encoding utf-8
-Sheet 1 2
+Sheet 1 3
 Title ""
 Date ""
@@
 $EndComp
 $Comp
-L Connector:RJ45_LED J?
-U 1 1 60AAB6B6
-P 2250 6900
-F 0 "J?" V 2296 6470 50  0000 R CNN
-F 1 "RJ45_LED" V 2205 6470 50  0000 R CNN
-F 2 "" V 2250 6925 50  0001 C CNN
-F 3 "~" V 2250 6925 50  0001 C CNN
-	1    2250 6900
-	0    -1   -1   0
-$EndComp
-$Comp
-L Connector:RJ45_LED J?
-U 1 1 60AAF3A4
-P 4100 6875
-F 0 "J?" V 4146 6445 50  0000 R CNN
-F 1 "RJ45_LED" V 4055 6445 50  0000 R CNN
-F 2 "" V 4100 6900 50  0001 C CNN
-F 3 "~" V 4100 6900 50  0001 C CNN
-	1    4100 6875
-	0    -1   -1   0
-$EndComp
-$Comp
-L Connector:USB_B J?
+L Connector:USB_B J1005
 U 1 1 60AB21AF
 P 9725 2800
-F 0 "J?" H 9782 3267 50  0000 C CNN
+F 0 "J1005" H 9782 3267 50  0000 C CNN
 F 1 "USB_B" H 9782 3176 50  0000 C CNN
-F 2 "" H 9875 2750 50  0001 C CNN
+F 2 "Connector_USB:USB_B_Amphenol_MUSB-D511_Vertical_Rugged" H 9875 2750 50  0001 C CNN
 F 3 " ~" H 9875 2750 50  0001 C CNN
 	1    9725 2800
@@
 $EndComp
 $Comp
-L Connector:USB_A J?
+L Connector:USB_A J1006
 U 1 1 60AB3DC4
 P 9725 4750
-F 0 "J?" H 9782 5217 50  0000 C CNN
+F 0 "J1006" H 9782 5217 50  0000 C CNN
 F 1 "USB_A" H 9782 5126 50  0000 C CNN
-F 2 "" H 9875 4700 50  0001 C CNN
+F 2 "Connector_USB:USB3_A_Molex_48393-001" H 9875 4700 50  0001 C CNN
 F 3 " ~" H 9875 4700 50  0001 C CNN
 	1    9725 4750
@@
 F1 "AudioToRpi.sch" 50
 $EndSheet
+$Sheet
+S 3550 1250 1300 1475
+U 60B0058A
+F0 "Audio-out" 50
+F1 "Audio-out.sch" 50
+$EndSheet
+$Comp
+L Connector:RJ12 J1003
+U 1 1 60B1A8BB
+P 2025 7100
+F 0 "J1003" V 2128 6770 50  0000 R CNN
+F 1 "RJ12" V 2037 6770 50  0000 R CNN
+F 2 "Connector_RJ:RJ12_Amphenol_54601" V 2025 7125 50  0001 C CNN
+F 3 "~" V 2025 7125 50  0001 C CNN
+	1    2025 7100
+	0    -1   -1   0
+$EndComp
+$Comp
+L Connector:RJ12 J1004
+U 1 1 60B1B236
+P 3575 7075
+F 0 "J1004" V 3678 6745 50  0000 R CNN
+F 1 "RJ12" V 3587 6745 50  0000 R CNN
+F 2 "Connector_RJ:RJ12_Amphenol_54601" V 3575 7100 50  0001 C CNN
+F 3 "~" V 3575 7100 50  0001 C CNN
+	1    3575 7075
+	0    -1   -1   0
+$EndComp
 $EndSCHEMATC

Commit message: PIC32MZ_EF_100
Connections:
- net labels added: BFE, BFR, BP1, BP2, HP, MICRO, PTT
- wire segments 80 -> 92
Changed lines of the file:
@@
 F0 "Audio-out" 50
 F1 "Audio-out.sch" 50
+F2 "FOSC" I L 3550 1400 50
+F3 "BFR" I L 3550 1875 50
+F4 "HP" I L 3550 1950 50
+F5 "DEMOD" I L 3550 1700 50
+F6 "CMD-TX" I L 3550 2325 50
+F7 "BFE" I R 4850 1650 50
+F8 "micro" I R 4850 1525 50
+F9 "CMD-RX" I L 3550 2425 50
 $EndSheet
 $Comp
@@
 	0    -1   -1   0
 $EndComp
+Wire Wire Line
+	2225 6700 2225 6525
+Text HLabel 2225 6525 1    50   Input ~ 0
+HP
+Text HLabel 2125 6525 1    50   Input ~ 0
+MICRO
+$Comp
+L power:GND #PWR?
+U 1 1 60F98169
+P 2025 6525
+F 0 "#PWR?" H 2025 6275 50  0001 C CNN
+F 1 "GND" H 2030 6352 50  0000 C CNN
+F 2 "" H 2025 6525 50  0001 C CNN
+F 3 "" H 2025 6525 50  0001 C CNN
+	1    2025 6525
+	-1   0    0    1
+$EndComp
+Text HLabel 1925 6525 1    50   Input ~ 0
+PTT
+Text HLabel 1825 6525 1    50   Input ~ 0
+BP1
+Text HLabel 1725 6525 1    50   Input ~ 0
+BP2
+Wire Wire Line
+	1725 6525 1725 6700
+Wire Wire Line
+	1825 6525 1825 6700
+Wire Wire Line
+	1925 6525 1925 6700
+Wire Wire Line
+	2025 6525 2025 6700
+Wire Wire Line
+	2125 6525 2125 6700
+Wire Wire Line
+	3775 6675 3775 6500
+Text HLabel 3775 6500 1    50   Input ~ 0
+BFR
+Text HLabel 3675 6500 1    50   Input ~ 0
+BFE
+$Comp
+L power:GND #PWR?
+U 1 1 60FAA332
+P 3575 6500
+F 0 "#PWR?" H 3575 6250 50  0001 C CNN
+F 1 "GND" H 3580 6327 50  0000 C CNN
+F 2 "" H 3575 6500 50  0001 C CNN
+F 3 "" H 3575 6500 50  0001 C CNN
+	1    3575 6500
+	-1   0    0    1
+$EndComp
+Text HLabel 3475 6500 1    50   Input ~ 0
+PTT
+Text HLabel 3375 6500 1    50   Input ~ 0
+BP1
+Text HLabel 3275 6500 1    50   Input ~ 0
+BP2
+Wire Wire Line
+	3275 6500 3275 6675
+Wire Wire Line
+	3375 6500 3375 6675
+Wire Wire Line
+	3475 6500 3475 6675
+Wire Wire Line
+	3575 6500 3575 6675
+Wire Wire Line
+	3675 6500 3675 6675
 $EndSCHEMATC

Commit message: CONNECTOR BOARD V2.00
Parts:
- removed J1005: USB_B, Connector_USB:USB_B_Amphenol_MUSB-D511_Vertical_Rugged, symbol Connector:USB_B
- removed J1006: USB_A, Connector_USB:USB3_A_Molex_48393-001, symbol Connector:USB_A
Connections:
- net labels added: CMD-RX, CMD-TX, DEMOD
- wire segments 92 -> 102
- no-connect marks 0 -> 2
Other:
- moved on the sheet: J1001, J1002
