File: Electronique/Audio/Audio IN_OUT/Audio-out.sch (KiCad schematic (older format))
At the start: 48 parts, among them Q3001 BSS123, U3001 MC33172, U3002 MF10, U3003 TDA2003

Commit message: MAJ
Parts:
- added C3020: 10µ, Capacitor_Tantalum_SMD:CP_EIA-3216-18_Kemet-A, symbol Device:CP
- C3003, C3010: value CP -> 10µ; footprint (none) -> Capacitor_Tantalum_SMD:CP_EIA-3216-18_Kemet-A
- C3011: value C -> 100n
- C3012: value CP -> 220µ; footprint (none) -> Capacitor_SMD:CP_Elec_6.3x5.4
- C3013: footprint (none) -> Capacitor_SMD:C_1210_3225Metric
- C3014: value CP -> 470µ; footprint (none) -> Capacitor_SMD:CP_Elec_6.3x3.9
- C3015: value C -> 47n
- C3016: footprint (none) -> Capacitor_Tantalum_SMD:CP_EIA-3216-18_Kemet-A
- C3017: value CP -> 1000µ; footprint (none) -> Capacitor_SMD:CP_Elec_6.3x4.9
- C3019: value C -> 0.1µ
- R3015: value R -> 100
- R3019: value R -> 47
- R3021: value R -> 220
- R3022: value R -> 2.2
- R3024: value R -> 1
Connections:
- net at Q3001.3 (D), R3015.1: now also C3020.2; no longer U3003.1 (+)
- new net: C3020.1, U3003.1 (+)
Other:
- moved on the sheet: C3009, C3010, R3015
Changed lines of the file:
@@
 L Device:CP C3010
 U 1 1 60B44FDA
-P 6800 2675
-F 0 "C3010" V 6545 2675 50  0000 C CNN
-F 1 "CP" V 6636 2675 50  0000 C CNN
-F 2 "" H 6838 2525 50  0001 C CNN
-F 3 "~" H 6800 2675 50  0001 C CNN
-	1    6800 2675
-	0    1    1    0
-$EndComp
-$Comp
-L Device:C C3015
-U 1 1 60B455B6
-P 9125 3525
-F 0 "C3015" V 8873 3525 50  0000 C CNN
-F 1 "C" V 8964 3525 50  0000 C CNN
-F 2 "Capacitor_SMD:C_0603_1608Metric" H 9163 3375 50  0001 C CNN
-F 3 "~" H 9125 3525 50  0001 C CNN
-	1    9125 3525
+P 6525 2675
+F 0 "C3010" V 6270 2675 50  0000 C CNN
+F 1 "10µ" V 6361 2675 50  0000 C CNN
+F 2 "Capacitor_Tantalum_SMD:CP_EIA-3216-18_Kemet-A" H 6563 2525 50  0001 C CNN
+F 3 "~" H 6525 2675 50  0001 C CNN
+	1    6525 2675
 	0    1    1    0
 $EndComp
@@
 P 8675 3525
 F 0 "R3019" V 8468 3525 50  0000 C CNN
-F 1 "R" V 8559 3525 50  0000 C CNN
+F 1 "47" V 8559 3525 50  0000 C CNN
 F 2 "Resistor_SMD:R_0603_1608Metric" V 8605 3525 50  0001 C CNN
 F 3 "~" H 8675 3525 50  0001 C CNN
@@
 P 9700 2975
 F 0 "R3021" H 9770 3021 50  0000 L CNN
-F 1 "R" H 9770 2930 50  0000 L CNN
+F 1 "220" H 9770 2930 50  0000 L CNN
 F 2 "Resistor_SMD:R_0603_1608Metric" V 9630 2975 50  0001 C CNN
 F 3 "~" H 9700 2975 50  0001 C CNN
@@
 P 9700 4100
 F 0 "R3022" H 9770 4146 50  0000 L CNN
-F 1 "R" H 9770 4055 50  0000 L CNN
+F 1 "2.2" H 9770 4055 50  0000 L CNN
 F 2 "Resistor_SMD:R_0603_1608Metric" V 9630 4100 50  0001 C CNN
 F 3 "~" H 9700 4100 50  0001 C CNN
@@
 P 8875 3850
 F 0 "C3014" V 9130 3850 50  0000 C CNN
-F 1 "CP" V 9039 3850 50  0000 C CNN
-F 2 "" H 8913 3700 50  0001 C CNN
+F 1 "470µ" V 9039 3850 50  0000 C CNN
+F 2 "Capacitor_SMD:CP_Elec_6.3x3.9" H 8913 3700 50  0001 C CNN
 F 3 "~" H 8875 3850 50  0001 C CNN
 	1    8875 3850
@@
 P 10075 2775
 F 0 "C3017" V 10330 2775 50  0000 C CNN
-F 1 "CP" V 10239 2775 50  0000 C CNN
-F 2 "" H 10113 2625 50  0001 C CNN
+F 1 "1000µ" V 10239 2775 50  0000 C CNN
+F 2 "Capacitor_SMD:CP_Elec_6.3x4.9" H 10113 2625 50  0001 C CNN
 F 3 "~" H 10075 2775 50  0001 C CNN
 	1    10075 2775
@@
 P 10400 2975
 F 0 "C3019" H 10515 3021 50  0000 L CNN
-F 1 "C" H 10515 2930 50  0000 L CNN
+F 1 "0.1µ" H 10515 2930 50  0000 L CNN
 F 2 "Capacitor_SMD:C_0603_1608Metric" H 10438 2825 50  0001 C CNN
 F 3 "~" H 10400 2975 50  0001 C CNN
@@
 P 10400 3375
 F 0 "R3024" H 10470 3421 50  0000 L CNN
-F 1 "R" H 10470 3330 50  0000 L CNN
+F 1 "1" H 10470 3330 50  0000 L CNN
 F 2 "Resistor_SMD:R_0603_1608Metric" V 10330 3375 50  0001 C CNN
 F 3 "~" H 10400 3375 50  0001 C CNN
@@
 L Device:C C3009
 U 1 1 60BB767E
-P 6800 2125
-F 0 "C3009" V 6548 2125 50  0000 C CNN
-F 1 "C" V 6639 2125 50  0000 C CNN
-F 2 "Capacitor_SMD:C_0603_1608Metric" H 6838 1975 50  0001 C CNN
-F 3 "~" H 6800 2125 50  0001 C CNN
-	1    6800 2125
-	0    1    1    0
-$EndComp
-Wire Wire Line
-	6950 2125 8075 2125
+P 6525 2125
+F 0 "C3009" V 6273 2125 50  0000 C CNN
+F 1 "C" V 6364 2125 50  0000 C CNN
+F 2 "Capacitor_SMD:C_0603_1608Metric" H 6563 1975 50  0001 C CNN
+F 3 "~" H 6525 2125 50  0001 C CNN
+	1    6525 2125
+	0    1    1    0
+$EndComp
+Wire Wire Line
+	6675 2125 8075 2125
 $Comp
 L Device:CP C3016
@@
 F 0 "C3016" V 9780 1725 50  0000 C CNN
 F 1 "10µ" V 9689 1725 50  0000 C CNN
-F 2 "" H 9563 1575 50  0001 C CNN
+F 2 "Capacitor_Tantalum_SMD:CP_EIA-3216-18_Kemet-A" H 9563 1575 50  0001 C CNN
 F 3 "~" H 9525 1725 50  0001 C CNN
 	1    9525 1725
@@
 F 0 "C3013" V 7925 1400 50  0000 C CNN
 F 1 "1µ" V 8025 1550 50  0000 C CNN
-F 2 "" H 8113 1275 50  0001 C CNN
+F 2 "Capacitor_SMD:C_1210_3225Metric" H 8113 1275 50  0001 C CNN
 F 3 "~" H 8075 1425 50  0001 C CNN
 	1    8075 1425
@@
 Connection ~ 5300 1475
 Wire Wire Line
-	5300 1100 6625 1100
+	5300 1100 6300 1100
 Wire Wire Line
 	5300 1475 5300 1100
@@
 F 1 "MF10" H 4775 1456 60  0000 C CNN
 F 2 "Package_SO:SOIC-20W_7.5x12.8mm_P1.27mm" H 4450 1475 60  0001 C CNN
-F 3 "http://www.onsemi.com/pub/Collateral/MC33171-D.PDF" H 4450 1475 60  0000 C CNN
+F 3 "http://www.onsemi.com/pub/Collateral/MC33171-D.PDF" H 4450 1475 60  0001 C CNN
 	1    4450 1475
 	1    0    0    -1
 $EndComp
 Wire Wire Line
-	6625 1100 6625 2125
+	6300 1100 6300 2125
 Wire Wire Line
 	10650 1725 11000 1725
@@
 	925  3375 1150 3375
 Wire Wire Line
-	6625 2125 6650 2125
+	6300 2125 6375 2125
 $Comp
 L Device:CP C3012
@@
 P 7925 2950
 F 0 "C3012" H 8043 2996 50  0000 L CNN
-F 1 "CP" H 8043 2905 50  0000 L CNN
-F 2 "" H 7963 2800 50  0001 C CNN
+F 1 "220µ" H 8043 2905 50  0000 L CNN
+F 2 "Capacitor_SMD:CP_Elec_6.3x5.4" H 7963 2800 50  0001 C CNN
 F 3 "~" H 7925 2950 50  0001 C CNN
 	1    7925 2950
@@
 P 7600 2950
 F 0 "C3011" H 7715 2996 50  0000 L CNN
-F 1 "C" H 7715 2905 50  0000 L CNN
+F 1 "100n" H 7715 2905 50  0000 L CNN
 F 2 "Capacitor_SMD:C_0603_1608Metric" H 7638 2800 50  0001 C CNN
 F 3 "~" H 7600 2950 50  0001 C CNN
@@
 	1    0    0    -1
 $EndComp
-Wire Wire Line
-	6625 2125 6625 2675
-Wire Wire Line
-	6625 2675 6650 2675
-Connection ~ 6625 2125
 $Comp
 L power:+BATT #PWR0136
@@
 P 3050 2025
 F 0 "C3003" V 3305 2025 50  0000 C CNN
-F 1 "CP" V 3214 2025 50  0000 C CNN
-F 2 "" H 3088 1875 50  0001 C CNN
+F 1 "10µ" V 3214 2025 50  0000 C CNN
+F 2 "Capacitor_Tantalum_SMD:CP_EIA-3216-18_Kemet-A" H 3088 1875 50  0001 C CNN
 F 3 "~" H 3050 2025 50  0001 C CNN
 	1    3050 2025
@@
 L Device:R R3015
 U 1 1 60E354FE
-P 7200 2675
-F 0 "R3015" V 6993 2675 50  0000 C CNN
-F 1 "R" V 7084 2675 50  0000 C CNN
-F 2 "Resistor_SMD:R_0603_1608Metric" V 7130 2675 50  0001 C CNN
-F 3 "~" H 7200 2675 50  0001 C CNN
-	1    7200 2675
+P 6850 2675
+F 0 "R3015" V 6643 2675 50  0000 C CNN
+F 1 "100" V 6734 2675 50  0000 C CNN
+F 2 "Resistor_SMD:R_0603_1608Metric" V 6780 2675 50  0001 C CNN
+F 3 "~" H 6850 2675 50  0001 C CNN
+	1    6850 2675
 	0    1    1    0
 $EndComp
@@
 $EndComp
 Wire Wire Line
-	7350 2675 7425 2675
-Wire Wire Line
-	6950 2675 7050 2675
-Wire Wire Line
-	7425 2675 7425 3050
-Wire Wire Line
-	7425 3050 7025 3050
-Wire Wire Line
-	7025 3050 7025 3125
-Connection ~ 7425 2675
-Wire Wire Line
-	7425 2675 8300 2675
+	7000 2675 7025 2675
+Wire Wire Line
+	6675 2675 6700 2675
 Wire Wire Line
 	7025 3525 7025 3600
@@
 Wire Wire Line
 	1100 2125 950  2125
+Wire Wire Line
+	7025 2675 7025 3125
+$Comp
+L Device:CP C3020
+U 1 1 60BA34C4
+P 7200 2675
+F 0 "C3020" V 6945 2675 50  0000 C CNN
+F 1 "10µ" V 7036 2675 50  0000 C CNN
+F 2 "Capacitor_Tantalum_SMD:CP_EIA-3216-18_Kemet-A" H 7238 2525 50  0001 C CNN
+F 3 "~" H 7200 2675 50  0001 C CNN
+	1    7200 2675
+	0    1    1    0
+$EndComp
+Wire Wire Line
+	6300 2125 6300 2675
+Wire Wire Line
+	6300 2675 6375 2675
+Connection ~ 6300 2125
+Wire Wire Line
+	7025 2675 7050 2675
+Connection ~ 7025 2675
+Wire Wire Line
+	7350 2675 8300 2675
+$Comp
+L Device:C C3015
+U 1 1 60B455B6
+P 9125 3525
+F 0 "C3015" V 8873 3525 50  0000 C CNN
+F 1 "47n" V 8964 3525 50  0000 C CNN
+F 2 "Capacitor_SMD:C_0603_1608Metric" H 9163 3375 50  0001 C CNN
+F 3 "~" H 9125 3525 50  0001 C CNN
+	1    9125 3525
+	0    1    1    0
+$EndComp
 $EndSCHEMATC

Commit message: PIC32MZ_EF_100
Parts:
- added C?: C, Capacitor_SMD:C_0603_1608Metric, symbol Device:C
- added C?: 10µ, Capacitor_Tantalum_SMD:CP_EIA-3216-18_Kemet-A, symbol Device:CP
- added C?: 1n, Capacitor_SMD:C_0603_1608Metric, symbol Device:C
- added C?: 1µ, Capacitor_SMD:C_1210_3225Metric, symbol Device:C
- added C? (x3): C, symbol Device:C
- added C? (x2): 100n, symbol Device:C
- added C?: 220p, symbol Device:C
- added L?: L, symbol Device:L
- added Q?: BC847, Package_TO_SOT_SMD:SOT-23, symbol Transistor_BJT:BC847
- added R? (x4): 100k, Resistor_SMD:R_0603_1608Metric, symbol Device:R
- added R?: 220, Resistor_SMD:R_0603_1608Metric, symbol Device:R
- added R?: 470, Resistor_SMD:R_0603_1608Metric, symbol Device:R
- added R? (x4): 100k, symbol Device:R
- added R?: R, symbol Device:R
- added R?: 680, symbol Device:R
- added R?: 22k, symbol Device:R
- added U? (x3): MC33172, symbol Amplifier_Operational:MC33172
Connections:
- net +5VA: now also C?.1, R?.1, R?.1, R?.1, U?.8 (V+)
- net GND: now also C?.1, C?.2, C?.2, C?.2, C?.2, C?.2, Q?.2 (E), R?.1, R?.2, U?.4 (V-)
- new net: C?.1, R?.1, U?.1
- new net: R?.1, R?.2, U?.2 (-)
- new net: C?.1, R?.1, R?.2, U?.3 (+)
- new net: C?.1, R?.2
- new net: C?.2, R?.2, U?.7
- new net: C?.2, R?.2 (x2)
- new net: C?.1, R?.1, R?.2
- new net: C?.2, R?.2, R?.2, U?.5 (+)
- new net: R?.1, R?.2, U?.6 (-)
- new net: C?.2, R?.1
- new net: C?.1, L?.1, R?.1, R?.2
- new net: C?.1, C?.1, Q?.3 (C)
- new net: C?.1, Q?.1 (B), R?.1
- new net BFE: R?.1
- new net CMD-RX: R?.2
- new net micro: L?.2

Commit message: CONNECTOR BOARD V2.00
Parts:
- removed C?: 220p, symbol Device:C
- removed Q?: BC847, Package_TO_SOT_SMD:SOT-23, symbol Transistor_BJT:BC847
- removed R?: 100k, symbol Device:R
- added Q201: BSS123, Package_TO_SOT_SMD:SOT-23, symbol Transistor_FET:BSS123
- C202, C206: renamed from C?; value C -> 100n; footprint (none) -> Capacitor_SMD:C_0603_1608Metric
- C204: renamed from C?; footprint Capacitor_SMD:C_1210_3225Metric -> Capacitor_SMD:C_0805_2012Metric
- C208, C209, C210: renamed from C?; footprint (none) -> Capacitor_SMD:C_0603_1608Metric
- L201: renamed from L?; footprint (none) -> Capacitor_SMD:C_1206_3216Metric
- R207, R208, R209, R210, R212, R213: renamed from R?; footprint (none) -> Resistor_SMD:R_0603_1608Metric
- U201: renamed from U?; footprint (none) -> Package_SO:SO-8_3.9x4.9mm_P1.27mm
- U3003: footprint CEN-PCB:TDA2003V -> Package_TO_SOT_THT:TO-220-5_P3.4x3.8mm_StaggerOdd_Lead7.13mm_TabDown
- gave numbers to parts that had none: 9
Connections:
- net CMD-RX: now also Q201.1 (G)
- net GND: now also Q201.2 (S)
- net at C208.1, C209.1: now also Q201.3 (D)
- net FOSC renamed OSC-MF10/FOSC
Other:
- moved on the sheet: C201, C202, C203, C204, C205, C206, C208, C209, C210, L201, R201, R202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
