File: Electronique/PIC32MXCubeV1/PIC32MXCubeV1/PIC32MX795F512L.sch (KiCad schematic (older format))
At the start: 25 parts, among them Q3003 2N7002, U2002 MCP1501, U2003 REF3020, U3004 PIC32MX795F512L, Y2001 Crystal_Small, Y2002 Crystal

Commit message: PIC32MZ_EF_100
Parts:
- C2003: value C -> NC
- R2002: value R -> 100
- R2004: value R -> 10k
- R3007: value R -> 1k
- R3008: value R -> 1k5
Changed lines of the file:
@@
 AR Path="/610AAB12/60977C74" Ref="R?"  Part="1"
 F 0 "R2004" H 1203 846 50  0000 L CNN
-F 1 "R" H 1203 755 50  0000 L CNN
+F 1 "10k" H 1203 755 50  0000 L CNN
 F 2 "Resistor_SMD:R_0603_1608Metric" H 1150 900 60  0001 C CNN
 F 3 "" H 1150 900 60  0000 C CNN
@@
 AR Path="/610AAB12/6097814A" Ref="R?"  Part="1"
 F 0 "R2002" V 2760 600 50  0000 C CNN
-F 1 "R" V 2851 600 50  0000 C CNN
+F 1 "100" V 2851 600 50  0000 C CNN
 F 2 "Resistor_SMD:R_0603_1608Metric" H 2950 700 60  0001 C CNN
 F 3 "" H 2950 700 60  0000 C CNN
@@
 AR Path="/610AAB12/60978786" Ref="C?"  Part="1"
 F 0 "C2003" H 1265 1471 50  0000 L CNN
-F 1 "C" H 1265 1380 50  0000 L CNN
+F 1 "NC" H 1265 1380 50  0000 L CNN
 F 2 "Capacitor_SMD:C_0603_1608Metric" H 1188 1275 50  0001 C CNN
 F 3 "~" H 1150 1425 50  0001 C CNN
@@
 P 8375 975
 F 0 "R3007" H 8445 1021 50  0000 L CNN
-F 1 "R" H 8445 930 50  0000 L CNN
+F 1 "1k" H 8445 930 50  0000 L CNN
 F 2 "Resistor_SMD:R_0603_1608Metric" V 8305 975 50  0001 C CNN
 F 3 "~" H 8375 975 50  0001 C CNN
@@
 P 8375 1400
 F 0 "R3008" H 8445 1446 50  0000 L CNN
-F 1 "R" H 8445 1355 50  0000 L CNN
+F 1 "1k5" H 8445 1355 50  0000 L CNN
 F 2 "Resistor_SMD:R_0603_1608Metric" V 8305 1400 50  0001 C CNN
 F 3 "~" H 8375 1400 50  0001 C CNN
