File: Electronique/PIC32MZ_EF_100_CubeV1/PIC32MZ_EF_100/I2C.sch (KiCad schematic (older format))
At the start: 21 parts, among them J3001 Conn_02x10_Odd_Even, Q3001 2N7002, Q3002 2N7002, U2001 PCF8563T, U3001 24LC1025, U3002 LM75A, U3003 SAA1064T, Y2003 Crystal

Commit message: PIC32MZ_EF_100
Parts:
- removed J3001: Conn_02x10_Odd_Even, Connector_PinHeader_1.27mm:PinHeader_2x10_P1.27mm_Vertical, symbol Connector_Generic:Conn_02x10_Odd_Even
- added C2008, C2009: 100n, Capacitor_SMD:C_0603_1608Metric, symbol Device:C
- added J2001, J2002: Conn_02x05_Top_Bottom, Connector_PinSocket_2.54mm:PinSocket_2x05_P2.54mm_Horizontal, symbol Connector_Generic:Conn_02x05_Odd_Even
- added Q2001, Q2002: BSR19, Package_TO_SOT_SMD:SOT-23, symbol Transistor_BJT:BC817
Connections:
- net labels added: A34, B34, C34, D34, E34, F34, G34, P34
- wire segments 134 -> 148
Other:
- moved on the sheet: C2004, C2007, R2003
