File: Electronique/ConnectorCubeV2/ConnectorCubeV2-A/IO.sch (KiCad schematic (older format))
At the start: 0 parts

Commit message: maj electronique
Parts:
- added J1003, J1004, J1005, J1006, J1007, J1008, J1009, J1010, J1011, J1012, J1013: Conn_01x03, Connector_JST:JST_GH_BM03B-GHS-TBT_1x03-1MP_P1.25mm_Vertical, symbol Connector_Generic:Conn_01x03
- added R1001, R1002, R1003, R1004, R1005, R1006, R1007, R1008, R1009, R1010, R1011, R1012, R1013, R1014, R1015, R1016, R1017, R1018, R1019, R1020, R1021, R1022: R, Resistor_SMD:R_0603_1608Metric, symbol Device:R
Connections:
- new net: J1003.2 (Pin_2), R1001.1, R1003.2
- new net: J1004.2 (Pin_2), R1002.1, R1004.2
- new net: J1005.2 (Pin_2), R1005.1, R1007.2
- new net: J1006.2 (Pin_2), R1006.1, R1008.2
- new net: J1007.2 (Pin_2), R1009.1, R1011.2
- new net: J1008.2 (Pin_2), R1010.1, R1012.2
- new net: J1009.2 (Pin_2), R1013.1, R1015.2
- new net: J1010.2 (Pin_2), R1014.1, R1016.2
- new net: J1011.2 (Pin_2), R1017.1, R1019.2
- new net: J1012.2 (Pin_2), R1018.1, R1020.2
- new net: J1013.2 (Pin_2), R1021.1, R1022.2
- new net +3V3: R1001.2, R1002.2, R1005.2, R1006.2, R1009.2, R1010.2, R1013.2, R1014.2, R1017.2, R1018.2, R1021.2
- new net +5VD: R1003.1, R1004.1, R1007.1, R1008.1, R1011.1, R1012.1, R1015.1, R1016.1, R1019.1, R1020.1, R1022.1
- new net GND: J1003.1 (Pin_1), J1004.1 (Pin_1), J1005.1 (Pin_1), J1006.1 (Pin_1), J1007.1 (Pin_1), J1008.1 (Pin_1), J1009.1 (Pin_1), J1010.1 (Pin_1), J1011.1 (Pin_1), J1012.1 (Pin_1), J1013.1 (Pin_1)
- new net IO0: J1003.3 (Pin_3)
- new net IO1: J1005.3 (Pin_3)
- new net IO10: J1013.3 (Pin_3)
- new net IO2: J1007.3 (Pin_3)
- new net IO3: J1009.3 (Pin_3)
- new net IO4: J1011.3 (Pin_3)
- new net IO5: J1004.3 (Pin_3)
- new net IO6: J1006.3 (Pin_3)
- new net IO7: J1008.3 (Pin_3)
- new net IO8: J1010.3 (Pin_3)
- new net IO9: J1012.3 (Pin_3)

Commit message: CONNECTOR BOARD V2.00
Parts:
- R1001, R1002, R1003, R1004, R1005, R1007, R1009, R1010, R1011, R1012, R1013, R1014, R1015, R1016, R1017, R1018, R1019, R1020, R1021, R1022: value R -> 0
Changed lines of the file:
@@
 $Descr A4 11693 8268
 encoding utf-8
-Sheet 10 10
+Sheet 10 12
 Title "Connector Cube V2"
-Date "2021-12-05"
+Date "2021-12-21"
 Rev "V2.00A"
 Comp "CubeDeb-F4DEB"
@@
 P 2325 2725
 F 0 "R1003" V 2118 2725 50  0000 C CNN
-F 1 "R" V 2209 2725 50  0000 C CNN
+F 1 "0" V 2209 2725 50  0000 C CNN
 F 2 "Resistor_SMD:R_0603_1608Metric" V 2255 2725 50  0001 C CNN
 F 3 "~" H 2325 2725 50  0001 C CNN
@@
 P 1925 2725
 F 0 "R1001" V 1718 2725 50  0000 C CNN
-F 1 "R" V 1809 2725 50  0000 C CNN
+F 1 "0" V 1809 2725 50  0000 C CNN
 F 2 "Resistor_SMD:R_0603_1608Metric" V 1855 2725 50  0001 C CNN
 F 3 "~" H 1925 2725 50  0001 C CNN
@@
 P 2325 3775
 F 0 "R1004" V 2118 3775 50  0000 C CNN
-F 1 "R" V 2209 3775 50  0000 C CNN
+F 1 "0" V 2209 3775 50  0000 C CNN
 F 2 "Resistor_SMD:R_0603_1608Metric" V 2255 3775 50  0001 C CNN
 F 3 "~" H 2325 3775 50  0001 C CNN
@@
 P 1925 3775
 F 0 "R1002" V 1718 3775 50  0000 C CNN
-F 1 "R" V 1809 3775 50  0000 C CNN
+F 1 "0" V 1809 3775 50  0000 C CNN
 F 2 "Resistor_SMD:R_0603_1608Metric" V 1855 3775 50  0001 C CNN
 F 3 "~" H 1925 3775 50  0001 C CNN
@@
 P 4100 2725
 F 0 "R1007" V 3893 2725 50  0000 C CNN
-F 1 "R" V 3984 2725 50  0000 C CNN
+F 1 "0" V 3984 2725 50  0000 C CNN
 F 2 "Resistor_SMD:R_0603_1608Metric" V 4030 2725 50  0001 C CNN
 F 3 "~" H 4100 2725 50  0001 C CNN
@@
 P 3700 2725
 F 0 "R1005" V 3493 2725 50  0000 C CNN
-F 1 "R" V 3584 2725 50  0000 C CNN
+F 1 "0" V 3584 2725 50  0000 C CNN
 F 2 "Resistor_SMD:R_0603_1608Metric" V 3630 2725 50  0001 C CNN
 F 3 "~" H 3700 2725 50  0001 C CNN
@@
 P 5900 2725
 F 0 "R1011" V 5693 2725 50  0000 C CNN
-F 1 "R" V 5784 2725 50  0000 C CNN
+F 1 "0" V 5784 2725 50  0000 C CNN
 F 2 "Resistor_SMD:R_0603_1608Metric" V 5830 2725 50  0001 C CNN
 F 3 "~" H 5900 2725 50  0001 C CNN
@@
 P 5500 2725
 F 0 "R1009" V 5293 2725 50  0000 C CNN
-F 1 "R" V 5384 2725 50  0000 C CNN
+F 1 "0" V 5384 2725 50  0000 C CNN
 F 2 "Resistor_SMD:R_0603_1608Metric" V 5430 2725 50  0001 C CNN
 F 3 "~" H 5500 2725 50  0001 C CNN
@@
 P 5900 3775
 F 0 "R1012" V 5693 3775 50  0000 C CNN
-F 1 "R" V 5784 3775 50  0000 C CNN
+F 1 "0" V 5784 3775 50  0000 C CNN
 F 2 "Resistor_SMD:R_0603_1608Metric" V 5830 3775 50  0001 C CNN
 F 3 "~" H 5900 3775 50  0001 C CNN
@@
 P 5500 3775
 F 0 "R1010" V 5293 3775 50  0000 C CNN
-F 1 "R" V 5384 3775 50  0000 C CNN
+F 1 "0" V 5384 3775 50  0000 C CNN
 F 2 "Resistor_SMD:R_0603_1608Metric" V 5430 3775 50  0001 C CNN
 F 3 "~" H 5500 3775 50  0001 C CNN
@@
 P 7675 2725
 F 0 "R1015" V 7468 2725 50  0000 C CNN
-F 1 "R" V 7559 2725 50  0000 C CNN
+F 1 "0" V 7559 2725 50  0000 C CNN
 F 2 "Resistor_SMD:R_0603_1608Metric" V 7605 2725 50  0001 C CNN
 F 3 "~" H 7675 2725 50  0001 C CNN
@@
 P 7275 2725
 F 0 "R1013" V 7068 2725 50  0000 C CNN
-F 1 "R" V 7159 2725 50  0000 C CNN
+F 1 "0" V 7159 2725 50  0000 C CNN
 F 2 "Resistor_SMD:R_0603_1608Metric" V 7205 2725 50  0001 C CNN
 F 3 "~" H 7275 2725 50  0001 C CNN
@@
 P 7675 3775
 F 0 "R1016" V 7468 3775 50  0000 C CNN
-F 1 "R" V 7559 3775 50  0000 C CNN
+F 1 "0" V 7559 3775 50  0000 C CNN
 F 2 "Resistor_SMD:R_0603_1608Metric" V 7605 3775 50  0001 C CNN
 F 3 "~" H 7675 3775 50  0001 C CNN
@@
 P 7275 3775
 F 0 "R1014" V 7068 3775 50  0000 C CNN
-F 1 "R" V 7159 3775 50  0000 C CNN
+F 1 "0" V 7159 3775 50  0000 C CNN
 F 2 "Resistor_SMD:R_0603_1608Metric" V 7205 3775 50  0001 C CNN
 F 3 "~" H 7275 3775 50  0001 C CNN
@@
 P 9400 2750
 F 0 "R1019" V 9193 2750 50  0000 C CNN
-F 1 "R" V 9284 2750 50  0000 C CNN
+F 1 "0" V 9284 2750 50  0000 C CNN
 F 2 "Resistor_SMD:R_0603_1608Metric" V 9330 2750 50  0001 C CNN
 F 3 "~" H 9400 2750 50  0001 C CNN
@@
 P 9000 2750
 F 0 "R1017" V 8793 2750 50  0000 C CNN
-F 1 "R" V 8884 2750 50  0000 C CNN
+F 1 "0" V 8884 2750 50  0000 C CNN
 F 2 "Resistor_SMD:R_0603_1608Metric" V 8930 2750 50  0001 C CNN
 F 3 "~" H 9000 2750 50  0001 C CNN
@@
 P 9400 3800
 F 0 "R1020" V 9193 3800 50  0000 C CNN
-F 1 "R" V 9284 3800 50  0000 C CNN
+F 1 "0" V 9284 3800 50  0000 C CNN
 F 2 "Resistor_SMD:R_0603_1608Metric" V 9330 3800 50  0001 C CNN
 F 3 "~" H 9400 3800 50  0001 C CNN
@@
 P 9000 3800
 F 0 "R1018" V 8793 3800 50  0000 C CNN
-F 1 "R" V 8884 3800 50  0000 C CNN
+F 1 "0" V 8884 3800 50  0000 C CNN
 F 2 "Resistor_SMD:R_0603_1608Metric" V 8930 3800 50  0001 C CNN
 F 3 "~" H 9000 3800 50  0001 C CNN
@@
 P 2325 5000
 F 0 "R1022" V 2118 5000 50  0000 C CNN
-F 1 "R" V 2209 5000 50  0000 C CNN
+F 1 "0" V 2209 5000 50  0000 C CNN
 F 2 "Resistor_SMD:R_0603_1608Metric" V 2255 5000 50  0001 C CNN
 F 3 "~" H 2325 5000 50  0001 C CNN
@@
 P 1925 5000
 F 0 "R1021" V 1718 5000 50  0000 C CNN
-F 1 "R" V 1809 5000 50  0000 C CNN
+F 1 "0" V 1809 5000 50  0000 C CNN
 F 2 "Resistor_SMD:R_0603_1608Metric" V 1855 5000 50  0001 C CNN
 F 3 "~" H 1925 5000 50  0001 C CNN
