File: Electronique/ConnectorCubeV2/ConnectorCubeV2-A/ConnectorCubeV2-A.sch (KiCad schematic (older format))
At the start: 2 parts, among them J1001 Conn_02x20_Odd_Even, J1002 Conn_02x20_Odd_Even

Commit message: maj electronique
Connections:
- net labels added: D[0..7], SCS
- wire segments 80 -> 124
Other:
- moved on the sheet: J1001, J1002

Commit message: CONNECTOR BOARD V2.00
Connections:
- net labels removed: SCS
- wire segments 124 -> 127
Changed lines of the file:
@@
 $Descr A4 11693 8268
 encoding utf-8
-Sheet 1 10
+Sheet 1 12
 Title "Connector Cube V2"
-Date "2021-12-06"
+Date "2021-12-21"
 Rev "V2.00A"
 Comp "CubeDeb-F4DEB"
@@
 Wire Wire Line
 	7650 2525 7350 2525
-Wire Wire Line
-	7650 2625 7350 2625
 Wire Wire Line
 	7650 2725 7350 2725
@@
 Text Label 7525 2525 2    50   ~ 0
 SDA1
-Text Label 7525 2625 2    50   ~ 0
-SDA2
 Text Label 7525 2725 2    50   ~ 0
 SDA3
@@
 F2 "SDA1" I L 1725 3525 50
 F3 "SCL1" I L 1725 3450 50
-F4 "SDL2" I L 1725 3725 50
-F5 "SCL2" I L 1725 3650 50
-F6 "SDA3" I L 1725 3925 50
-F7 "SCL3" I L 1725 3850 50
+F4 "SCL2" I L 1725 3650 50
+F5 "SDA3" I L 1725 3925 50
+F6 "SCL3" I L 1725 3850 50
+F7 "SDA2" I L 1725 3725 50
 $EndSheet
 $Sheet
@@
 SCK1
 Text Label 3300 4825 0    50   ~ 0
-SCS
+IO10
 Text Label 3300 4900 0    50   ~ 0
 CS1
@@
 Wire Wire Line
 	2650 5650 2825 5650
+Text Label 2700 5650 0    50   ~ 0
+RST
+$Sheet
+S 7975 3475 775  1150
+U 61BE7334
+F0 "7Seg" 50
+F1 "7Seg.sch" 50
+F2 "CS7" I L 7975 3650 50
+F3 "CLK7" I L 7975 3750 50
+F4 "DIO7" I L 7975 3850 50
+$EndSheet
+Wire Wire Line
+	7825 3650 7975 3650
+Wire Wire Line
+	7825 3750 7975 3750
+Wire Wire Line
+	7825 3850 7975 3850
+Text Label 7825 3650 0    50   ~ 0
+IO5
+Text Label 7825 3750 0    50   ~ 0
+IO6
+Text Label 7825 3850 0    50   ~ 0
+IO7
+Text Label 7525 2625 2    50   ~ 0
+SDA2
+Wire Wire Line
+	7350 2625 7650 2625
 Wire Bus Line
 	7250 1725 7250 2100
 Wire Bus Line
 	8475 1625 8475 1975
-Text Label 2700 5650 0    50   ~ 0
-RST
+$Sheet
+S 8125 5525 500  700
+U 61C2E239
+F0 "POWER" 50
+F1 "Power.sch" 50
+$EndSheet
 $EndSCHEMATC
