File: Electronique/ConnectorCubeV2/ConnectorCubeV2-A/LCD.sch (KiCad schematic (older format))
At the start: 13 parts, among them J301 Conn_02x08_Odd_Even, J302 Conn_02x10_Odd_Even, Q301 BSS123, Q302 BSS123, Q303 BSS123, Q304 BSS123, Q305 BS250, U301 74LVCC3245

Commit message: V206 TM1638 7Segments Begin
Parts:
- U301: footprint Package_SO:SSOP-24_5.3x8.2mm_P0.65mm -> Package_SO:SSOP-24_3.9x8.7mm_P0.635mm
Changed lines of the file:
@@
 F 0 "U301" H 3250 4287 60  0000 C CNN
 F 1 "74LVCC3245" H 3250 4181 60  0000 C CNN
-F 2 "Package_SO:SSOP-24_5.3x8.2mm_P0.65mm" H 2950 4200 60  0001 C CNN
+F 2 "Package_SO:SSOP-24_3.9x8.7mm_P0.635mm" H 2950 4200 60  0001 C CNN
 F 3 "" H 2950 4200 60  0000 C CNN
 	1    2950 4200
