File: Electronique/Audio/Audio IN_OUT/V2.00/OSC-MF10.sch (KiCad schematic (older format))
At the start: 10 parts, among them U301 74LVC1G80, U302 PCF8574, U303 74HC4059, U304 MAX7375AXR805

Commit message: AUDIO BOARD V2-00
Parts:
- added Q305: BSS123, Package_TO_SOT_SMD:SOT-23, symbol Transistor_FET:BSS123
- added R313: R, Resistor_SMD:R_0603_1608Metric, symbol Device:R
Connections:
- net +5VD: now also R313.1; no longer U302.16 (VDD), U303.24 (VCC), U304.1 (V+)
- net FOSC: now also Q305.3 (D), R313.2; no longer U301.1 (D), U301.4 (~Q)
- net GND: now also Q305.2 (S)
- net +5VA renamed +3V3
- net +3V3: now also U302.16 (VDD), U303.24 (VCC), U304.1 (V+)
- new net: Q305.1 (G), U301.1 (D), U301.4 (~Q)
Changed lines of the file:
@@
 	9025 4075 9025 4150
-$Comp
-L power:+5VA #PWR0153
-U 1 1 61EE668F
-P 9025 3600
-F 0 "#PWR0153" H 9025 3450 50  0001 C CNN
-F 1 "+5VA" H 9040 3773 50  0000 C CNN
-F 2 "" H 9025 3600 50  0001 C CNN
-F 3 "" H 9025 3600 50  0001 C CNN
-	1    9025 3600
-	1    0    0    -1
-$EndComp
 $Comp
 L power:GND #PWR0164
@@
 	7825 3125 7825 3050
 $Comp
-L power:+5VD #PWR0168
-U 1 1 61C6F863
-P 7625 3050
-F 0 "#PWR0168" H 7625 2900 50  0001 C CNN
-F 1 "+5VD" H 7640 3223 50  0000 C CNN
-F 2 "" H 7625 3050 50  0001 C CNN
-F 3 "" H 7625 3050 50  0001 C CNN
-	1    7625 3050
-	1    0    0    -1
-$EndComp
-$Comp
 L power:GND #PWR0169
 U 1 1 61C6FE2E
@@
 Wire Wire Line
 	6050 3475 6050 3400
-$Comp
-L power:+5VD #PWR0171
-U 1 1 61C79E33
-P 6050 3400
-F 0 "#PWR0171" H 6050 3250 50  0001 C CNN
-F 1 "+5VD" H 6065 3573 50  0000 C CNN
-F 2 "" H 6050 3400 50  0001 C CNN
-F 3 "" H 6050 3400 50  0001 C CNN
-	1    6050 3400
-	1    0    0    -1
-$EndComp
 Wire Wire Line
 	6050 4875 6050 4950
@@
 	9350 3825 9700 3825
 Connection ~ 9350 3825
-Text HLabel 9700 3825 2    50   Input ~ 0
+Text HLabel 10275 3575 2    50   Input ~ 0
 FOSC
 NoConn ~ 5550 4575
@@
 	1    0    0    -1
 $EndComp
-$Comp
-L power:+5VD #PWR0178
-U 1 1 61CB5405
+Wire Wire Line
+	8675 3675 9350 3675
+Wire Wire Line
+	9025 3600 9025 3775
+$Comp
+L power:+3V3 #PWR0153
+U 1 1 62287274
+P 6050 3400
+F 0 "#PWR0153" H 6050 3250 50  0001 C CNN
+F 1 "+3V3" H 6065 3573 50  0000 C CNN
+F 2 "" H 6050 3400 50  0001 C CNN
+F 3 "" H 6050 3400 50  0001 C CNN
+	1    6050 3400
+	1    0    0    -1
+$EndComp
+$Comp
+L power:+3V3 #PWR0168
+U 1 1 62289C96
+P 7625 3050
+F 0 "#PWR0168" H 7625 2900 50  0001 C CNN
+F 1 "+3V3" H 7640 3223 50  0000 C CNN
+F 2 "" H 7625 3050 50  0001 C CNN
+F 3 "" H 7625 3050 50  0001 C CNN
+	1    7625 3050
+	1    0    0    -1
+$EndComp
+$Comp
+L power:+3V3 #PWR0171
+U 1 1 6228B563
 P 8425 5125
-F 0 "#PWR0178" H 8425 4975 50  0001 C CNN
-F 1 "+5VD" H 8440 5298 50  0000 C CNN
+F 0 "#PWR0171" H 8425 4975 50  0001 C CNN
+F 1 "+3V3" H 8440 5298 50  0000 C CNN
 F 2 "" H 8425 5125 50  0001 C CNN
 F 3 "" H 8425 5125 50  0001 C CNN
@@
 	1    0    0    -1
 $EndComp
-Wire Wire Line
-	8675 3675 9350 3675
-Wire Wire Line
-	9025 3600 9025 3775
+$Comp
+L power:+3V3 #PWR0178
+U 1 1 6228C644
+P 9025 3600
+F 0 "#PWR0178" H 9025 3450 50  0001 C CNN
+F 1 "+3V3" H 9040 3773 50  0000 C CNN
+F 2 "" H 9025 3600 50  0001 C CNN
+F 3 "" H 9025 3600 50  0001 C CNN
+	1    9025 3600
+	1    0    0    -1
+$EndComp
+$Comp
+L Transistor_FET:BSS123 Q305
+U 1 1 62293412
+P 9900 3825
+F 0 "Q305" H 10104 3871 50  0000 L CNN
+F 1 "BSS123" H 10104 3780 50  0000 L CNN
+F 2 "Package_TO_SOT_SMD:SOT-23" H 10100 3750 50  0001 L CIN
+F 3 "http://www.diodes.com/assets/Datasheets/ds30366.pdf" H 9900 3825 50  0001 L CNN
+	1    9900 3825
+	1    0    0    -1
+$EndComp
+$Comp
+L power:GND #PWR0190
+U 1 1 62296DF3
+P 10000 4100
+F 0 "#PWR0190" H 10000 3850 50  0001 C CNN
+F 1 "GND" H 10005 3927 50  0000 C CNN
+F 2 "" H 10000 4100 50  0001 C CNN
+F 3 "" H 10000 4100 50  0001 C CNN
+	1    10000 4100
+	1    0    0    -1
+$EndComp
+Wire Wire Line
+	10000 4025 10000 4100
+Wire Wire Line
+	10275 3575 10000 3575
+Wire Wire Line
+	10000 3575 10000 3625
+Wire Wire Line
+	10000 3575 10000 3475
+Connection ~ 10000 3575
+$Comp
+L Device:R R313
+U 1 1 622A0E76
+P 10000 3325
+F 0 "R313" H 10070 3371 50  0000 L CNN
+F 1 "R" H 10070 3280 50  0000 L CNN
+F 2 "Resistor_SMD:R_0603_1608Metric" V 9930 3325 50  0001 C CNN
+F 3 "~" H 10000 3325 50  0001 C CNN
+	1    10000 3325
+	1    0    0    -1
+$EndComp
+Wire Wire Line
+	10000 3175 10000 3100
+$Comp
+L power:+5VD #PWR0191
+U 1 1 622A3126
+P 10000 3100
+F 0 "#PWR0191" H 10000 2950 50  0001 C CNN
+F 1 "+5VD" H 10015 3273 50  0000 C CNN
+F 2 "" H 10000 3100 50  0001 C CNN
+F 3 "" H 10000 3100 50  0001 C CNN
+	1    10000 3100
+	1    0    0    -1
+$EndComp
 $EndSCHEMATC
