File: Electronique/Audio/Audio IN_OUT/V2.00/Audio IN_OUT.kicad_pcb (KiCad board)
At the start: 2 copper layers, 95.2 x 95.3 mm, 114 parts, among them J1001 Conn_02x20_Odd_Even, J1002 Conn_02x20_Odd_Even, J1003 RJ12, J1004 RJ12, J101 Conn_Coaxial, J102 Conn_Coaxial, J103 Conn_Coaxial, J104 Conn_Coaxial, Q201 BSS123, Q3001 BSS123, Q301 BSS123, Q302 BC807W, Q303 BC847, Q304 BC807W, Q305 BSS123, Q401 BSS123, Q402 BSS123, U201 MC33172, U202 MCP45HV51-ST, U3001 MC33172, U3002 MF10, U3003 TDA2003, U301 74LVC1G80, U302 PCF8574, U303 74HC4059, U304 MAX7375AXR805

Commit message: reprise 28-7-2022
Other:
- net class Default removed
