File: Electronique/CpuCubeV2/CpuCubeV2-00/I2C.kicad_sch (KiCad schematic)
At the start: 26 parts

Commit message: CPU CUBE V2-00
Parts:
- removed C2004: ~, symbol PIC32MZ_EF_100-rescue:CP-Device
- removed C2005, C2006, C2007, C2008, C2009, C3001: ~, symbol Device:C
- removed D2001: ~, symbol Device:D_Schottky
- removed J2001, J2002: ~, symbol Connector_Generic:Conn_02x05_Odd_Even
- removed Q2001, Q2002: ~, symbol Transistor_BJT:BC817
- removed Q3001, Q3002: ~, symbol Transistor_FET:2N7002
- removed R2003, R2005, R2006, R3001, R3002, R3003, R3004: ~, symbol Device:R
- removed U2001: ~, symbol Timer_RTC:PCF8563T
- removed U3001: ~, symbol Memory_EEPROM:24LC1025
- removed U3002: ~, symbol Sensor_Temperature:LM75C
- removed U3003: ~, symbol CEN-SCHEMA:SAA1064T
- removed Y2003: ~, symbol Device:Crystal
- added C? (x6): ~, symbol Device:C
- added C?: ~, symbol PIC32MZ_EF_100-rescue:CP-Device
- added D?: ~, symbol Device:D_Schottky
- added J? (x2): ~, symbol Connector_Generic:Conn_02x05_Odd_Even
- added Q? (x2): ~, symbol Transistor_FET:2N7002
- added Q? (x2): ~, symbol Transistor_BJT:BC817
- added R? (x7): ~, symbol Device:R
- added U?: ~, symbol Memory_EEPROM:24LC1025
- added U?: ~, symbol Timer_RTC:PCF8563T
- added U?: ~, symbol CEN-SCHEMA:SAA1064T
- added U?: ~, symbol Sensor_Temperature:LM75C
- added Y?: ~, symbol Device:Crystal
Connections:
- net +3V3: now also C?.1, C?.1, D?.2 (A), Q?.1 (G), Q?.1 (G), R?.1, R?.1, U?.8 (+Vs), U?.8 (VCC)
- net +5VD: now also C?.1, Q?.3 (C), Q?.3 (C), R?.1, R?.1, U?.13 (VCC)
- net A34: now also J?.7 (Pin_7), U?.17 (P11)
- net B34: now also J?.5 (Pin_5), U?.15 (P9)
- net C34: now also J?.6 (Pin_6), U?.18 (P12)
- net D34: now also J?.4 (Pin_4), U?.20 (P14)
- net E34: now also J?.2 (Pin_2), U?.19 (P13)
- net F34: now also J?.1 (Pin_1), U?.22 (P16)
- net G34: now also J?.8 (Pin_8), U?.21 (P15)
- net GND: now also C?.2, C?.2, C?.2, C?.2, C?.2, C?.2, U?.1 (A0), U?.1 (ADR), U?.12 (VSS), U?.2 (A1), U?.3 (A2), U?.4 (GND), U?.4 (GND), U?.4 (VSS), U?.5 (A2), U?.6 (A1), U?.7 (A0)
- net INT0: now also R?.1, R?.1
- net P34: now also J?.10 (Pin_10), U?.16 (P10)
- net SCL1: now also Q?.2 (S), R?.2, U?.2 (SCL), U?.6 (SCL), U?.6 (SCL)
- net SDA1: now also Q?.2 (S), R?.2, U?.1 (SDA), U?.5 (SDA), U?.5 (SDA)
- new net: J?.1 (Pin_1), U?.3 (P8)
- new net: J?.10 (Pin_10), U?.9 (P2)
- new net: J?.2 (Pin_2), U?.6 (P5)
- new net: J?.3 (Pin_3), J?.3 (Pin_3), Q?.2 (E)
- new net: J?.4 (Pin_4), U?.5 (P6)
- new net: J?.5 (Pin_5), U?.10 (P1)
- new net: J?.6 (Pin_6), U?.7 (P4)
- new net: J?.7 (Pin_7), U?.8 (P3)
- new net: J?.8 (Pin_8), U?.4 (P7)
- new net: J?.9 (Pin_9), J?.9 (Pin_9), Q?.2 (E)
- new net: Q?.3 (D), R?.2, U?.23 (SDA)
- new net: C?.1, U?.1 (OSCI), Y?.1
- new net: C?.1, D?.1 (K), R?.1, U?.8 (VDD)
- new net: U?.2 (OSCO), Y?.2
- new net: R?.2, U?.3 (O.S.)
- new net: R?.2, U?.3 (~{INT})
- new net: Q?.1 (B), U?.11 (MX1)
- new net: Q?.1 (B), U?.14 (MX2)
- new net: C?.1, U?.2 (CEXT)
- new net: Q?.3 (D), R?.2, U?.24 (SCL)
