File: Electronique/PIC32MX795F512L/PIC32MX795F512L/PIC32MX795F512L.kicad_sch (KiCad schematic)
At the start: 24 parts, among them J101 Conn_02x13_Odd_Even, J102 Conn_02x13_Odd_Even, J103 Conn_02x13_Odd_Even, J104 Conn_02x13_Odd_Even, U101 PIC32MX795F512L, Y101 8Mhz, Y102 Crystal_Small

Commit message: CPU CUBE V2-00
Parts:
- removed Y101: 8Mhz, Crystal:Crystal_SMD_HC49-SD, symbol Device:Crystal_Small
- added D1001: LED, Diode_SMD:D_0603_1608Metric, symbol Device:LED
- added R1001: 330, Resistor_SMD:R_0603_1608Metric, symbol Device:R
- added Y1001: 8Mhz, Crystal:Crystal_SMD_Abracon_ABM3C-4Pin_5.0x3.2mm, symbol Device:Crystal_GND24_Small
- C112: footprint Capacitor_Tantalum_SMD:CP_EIA-1608-08_AVX-J -> Capacitor_Tantalum_SMD:CP_EIA-3216-10_Kemet-I
- Y102: symbol Device:Crystal_Small -> Device:Crystal_GND23
Connections:
- net +3V3: now also D1001.2 (A)
- net 63: now also C101.1, R101.1, U101.63 (OSC1/CLKI/RC12), Y1001.1
- net 64: now also C103.1, R101.2, U101.64 (OSC2/CLKO/RC15), Y1001.3
- net 73: now also C102.1, U101.73 (SOSCI/CN1/RC13), Y102.4
- net 74: now also R102.1, U101.74 (SOSCO/T1CK/CN0/RC14)
- net 85: now also C105.1, U101.85 (VCAP/VDDCORE)
- net GND: now also R1001.2, Y1001.2, Y1001.4
- net at C104.1, R102.2: now also Y102.1; no longer Y102.2
- new net: D1001.1 (K), R1001.1
- no-connect marks 0 -> 2
Other:
- company: (none) -> F4DEB
- title: (none) -> PIC32MX795F512L-80I/PF
- moved on the sheet: C101, C102, C103, C104
