File: Electronique/PIC32MZ_EF_100_CubeV1/PIC32MZ_EF_100V2-00/PIC32MZ2048EF100.kicad_sch (KiCad schematic)
At the start: 47 parts

Commit message: CPU CUBE V2-00
Parts:
- 47µ3001, C2001, C2002, C2003, C3002, C3003, C3004, C3005, C3006, C3007, C3008, C3009, C3010, C3011, C3012, C3013, L3001, Q3003, R3005, R3006, R3007, R3008, R3009, R3010, R3011, R3012, R3013, R3014, R3015, R3016, R3017, R3018, R3019, R3020, R3021, R3022, R3023, R3024, R3025, R3026, R3027, R3028, R3029, U2002, U3004, X3001, Y2001: value (none) -> ~
